Commit message: feat: 新增ranger_mini机器人底盘URDF/XACRO模型与gazebo仿真配置
添加了完整的四轮转向移动底盘的连杆、关节定义，包含碰撞检测、视觉外观与惯性参数，新增ranger_mini.xacro完整描述文件，同时更新了原urdf文件的关节连接关系以适配新的底盘结构

File: autorunner_description/urdf/u1_arm/u1_arm_gazebo.urdf (robot description, URDF)
Before this commit: robot u1_arm, 8 links, 7 joints
Links:
- added link base_link, mass 10; collision box size=0.5 0.35 0.2; visual mesh filename=package://u1_arm_description/meshes/u1_arm/dae/ranger_base.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 scale=1 1 1
- added link fl_steering_wheel_link, mass 1; collision cylinder length=0.001 radius=0.001; visual mesh filename=package://u1_arm_description/meshes/u1_arm/dae/steering_whe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 scale=10 10 10
- added link fl_wheel_link, mass 8; collision cylinder length=0.08 radius=0.09; visual mesh filename=package://u1_arm_description/meshes/u1_arm/dae/wheel_v3.dae scale=10 10 10
- added link fr_steering_wheel_link, mass 1; collision cylinder length=0.001 radius=0.001; visual mesh filename=package://u1_arm_description/meshes/u1_arm/dae/steering_whe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 scale=10 10 10
- added link fr_wheel_link, mass 8; collision cylinder length=0.08 radius=0.09; visual mesh filename=package://u1_arm_description/meshes/u1_arm/dae/wheel_v3.dae scale=10 10 10
- added link rl_steering_wheel_link, mass 1; collision cylinder length=0.001 radius=0.001; visual mesh filename=package://u1_arm_description/meshes/u1_arm/dae/steering_whe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 scale=10 10 10
- added link rl_wheel_link, mass 8; collision cylinder length=0.08 radius=0.09; visual mesh filename=package://u1_arm_description/meshes/u1_arm/dae/wheel_v3.dae scale=10 10 10
- added link rr_steering_wheel_link, mass 1; collision cylinder length=0.001 radius=0.001; visual mesh filename=package://u1_arm_description/meshes/u1_arm/dae/steering_whe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 scale=10 10 10
- added link rr_wheel_link, mass 8; collision cylinder length=0.08 radius=0.09; visual mesh filename=package://u1_arm_description/meshes/u1_arm/dae/wheel_v3.dae scale=10 10 10
Joints:
- removed joint world_to_u1_frame
- added joint base_link_to_u1_frame: type fixed, parent base_link, child u1_frame, origin xyz=0.3275 -0.245 0.519 rpy=0 0 0
- added joint fl_steering_joint: type revolute, parent base_link, child fl_steering_wheel_link, origin xyz=0.25 0.19 -0.1 rpy=0 0 0, axis 0 0 -1, limit lower=-2.1 upper=2.1 effort=5 velocity=6.28
- added joint fl_wheel: type continuous, parent fl_steering_wheel_link, child fl_wheel_link, origin xyz=0.0 0.0 -0.12 rpy=0 0 0, axis 0 1 0
- added joint fr_steering_joint: type revolute, parent base_link, child fr_steering_wheel_link, origin xyz=0.25 -0.19 -0.1 rpy=0 0 0, axis 0 0 -1, limit lower=-2.1 upper=2.1 effort=5 velocity=6.28
- added joint fr_wheel: type continuous, parent fr_steering_wheel_link, child fr_wheel_link, origin xyz=0.0 0.0 -0.12 rpy=0 0 0, axis 0 1 0
- added joint rl_steering_joint: type revolute, parent base_link, child rl_steering_wheel_link, origin xyz=-0.25 0.19 -0.1 rpy=0 0 0, axis 0 0 -1, limit lower=-2.1 upper=2.1 effort=5 velocity=6.28
- added joint rl_wheel: type continuous, parent rl_steering_wheel_link, child rl_wheel_link, origin xyz=0.0 0.0 -0.12 rpy=0 0 0, axis 0 1 0
- added joint rr_steering_joint: type revolute, parent base_link, child rr_steering_wheel_link, origin xyz=-0.23 -0.206 -0.1 rpy=0 0 0, axis 0 0 -1, limit lower=-2.1 upper=2.1 effort=5 velocity=6.28
- added joint rr_wheel: type continuous, parent rr_steering_wheel_link, child rr_wheel_link, origin xyz=0.0 0.0 -0.12 rpy=0 0 0, axis 0 1 0
- added joint world_to_base_link: type fixed, parent world, child base_link, origin xyz=-0.3275 0.245 -0.519 rpy=0 0 0
