Commit message: fix(urdf): 替换u1_arm的mesh文件为u2.stl
将gazebo仿真urdf里的u1.stl替换为新增的u2.stl.7z网格文件

File: autorunner_description/urdf/AutoRunner/autorunner_gazebo.urdf (robot description, URDF)
Before this commit: robot autorunner, 11 links, 10 joints
Links:
- link u1_frame: geometry collision mesh filename=package://autorunner_description/meshes/AutoRunner/u2.stl scale=0.001 0.001 0.001; visual mesh filename=package://autorunner_description/meshes/AutoRunner/u2.stl scale=0.001 0.001 0.001

Commit message: fix(urdf+meshes): 更新机械臂关节l6和对应网格文件
1.  新增了l6连杆及固定关节j6到u1_arm的urdf文件
2.  替换了主体urdf的参考网格文件为u1.stl
3.  更新了u1_arm所有关节的STL网格文件

File: autorunner_description/urdf/AutoRunner/autorunner_gazebo.urdf (robot description, URDF)
Before this commit: robot autorunner, 11 links, 10 joints
Links:
- link u1_frame: geometry collision mesh filename=package://autorunner_description/meshes/AutoRunner/u1.stl scale=0.001 0.001 0.001; visual mesh filename=package://autorunner_description/meshes/AutoRunner/u1.stl scale=0.001 0.001 0.001

File: autorunner_description/urdf/u1_arm/u1_arm_gazebo.urdf (robot description, URDF)
Before this commit: robot u1_arm, 17 links, 16 joints
Links:
- added link l6, mass 0; collision mesh filename=package://u1_arm_description/meshes/u1_arm/l6.STL; visual mesh filename=package://u1_arm_description/meshes/u1_arm/l6.STL
Joints:
- added joint j6: type fixed, parent l5, child l6, origin xyz=0.15 0 0.011 rpy=-1.5708 0 -1.5708
